File: 6502.kicad_pcb (KiCad board)
At the start: 2 copper layers, 190.5 x 124.5 mm, 8 parts, among them U1 W65C02, U2 W65C22, U3 28C256, U4 62256, U5 W65C22, U6 ATF22V10

Commit message: Updated schematic design files
Parts:
- added J1: Barrel_Jack_Switch, Connector_BarrelJack:BarrelJack_Wuerth_6941xx301002, F.Cu at (43.2, 79.4)
- added R1: 1k, Resistor_THT:R_Axial_DIN0207_L6.3mm_D2.5mm_P7.62mm_Horizontal, F.Cu at (53.3, 67.3)
- added X1: ACO-xxxMHz, Oscillator:Oscillator_DIP-14, F.Cu at (41.9, 100.3)
Connections:
- U1 pad 2: unconnected-(U1-RDY-Pad2) -> Net-(U1-RDY)
- U1 pad 36: unconnected-(U1-BE-Pad36) -> +5V
- U1 pad 37: unconnected-(U1-ϕ0-Pad37) -> Net-(U1-ϕ0)
- U2 pad 25: unconnected-(U2-ϕ2-Pad25) -> Net-(U1-ϕ0)
- U5 pad 25: unconnected-(U5-ϕ2-Pad25) -> Net-(U1-ϕ0)
- U6 pad 1: unconnected-(U6-CLK/IN-Pad1) -> Net-(U1-ϕ0)
- U6 pad 12: unconnected-(U6-GND-Pad12) -> GND
- U6 pad 24: unconnected-(U6-VCC-Pad24) -> +5V
Routing:
- net Net-(U1-ϕ0): track 0.00 -> 159.7 mm
- net +5V: track 209.8 -> 321.0 mm, vias 1 -> 0
- net ~{OE}: track 164.0 -> 109.2 mm, vias 1 -> 0
- net GND: track 252.5 -> 306.3 mm
- net Net-(U1-RDY): track 0.00 -> 53.3 mm
- net /A5: track 176.2 -> 147.1 mm
- net /A7: track 150.8 -> 179.7 mm, vias 1 -> 0
- net Net-(U1-R/~{W}): track 138.2 -> 111.3 mm, vias 3 -> 0
- net /A11: track 159.1 -> 132.9 mm
- net /A13: track 126.0 -> 151.0 mm, vias 1 -> 0
- net /A6: track 169.9 -> 147.0 mm
- net /A12: track 175.2 -> 152.6 mm, vias 0 -> 1
- net /A3: track 186.0 -> 201.3 mm
- net ~{ROM}: track 82.9 -> 71.2 mm, vias 2 -> 0
- net ~{IO2}: track 88.4 -> 79.1 mm, vias 2 -> 1
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